Commit message: Commit for tdot_testcase

File: urdf/amr_arm_robot.xacro (robot description, xacro)
@@ -14,7 +14,7 @@
     <xacro:include filename="$(find herox_description)/urdf/herox_amr.urdf.xacro"/>
     <joint name="amr_arm_joint" type="fixed">
-	<origin xyz="0 0 0" rpy="0 0 0 "/>
-	<parent link="base_link"/>
-	<child link="base"/>
+      <origin xyz="0 0 0.395" rpy="0 0 0 "/>
+      <parent link="base_link"/>
+      <child link="base"/>
     </joint>
 </robot>
